File: MysXLedDimmer.sch (KiCad schematic (older format))
At the start: 8 parts, among them P1 MYSX_1.3, P2 CONN_01X02, P3 CONN_01X02, P4 CONN_01X02, Q1 IRLZ44N, Q2 IRLZ44N

Commit message: Changed to use IRLML2502 in sot23
Parts:
- added C1: C, Capacitors_SMD:C_0805_HandSoldering, symbol C
- added C2: CP, Capacitors_SMD:C_0805_HandSoldering, symbol CP
- added R3, R4: 27, Resistors_SMD:R_0805_HandSoldering, symbol R
- P1: value MYSX_1.3 -> MYSX_2.4; symbol MYSX_1.3 -> MYSX_2.3
- Q1, Q2: value IRLZ44N -> IRLML2502; footprint TO_SOT_Packages_THT:TO-220_Neutral123_Vertical -> TO_SOT_Packages_SMD:SOT-23_Handsoldering; symbol Q_PMOS_GDS -> Q_NMOS_GSD
- R1, R2: value 2k2 -> 100k
Connections:
- net +12V: now also C1.1, C2.1
- net GND: now also Q1.2 (S), Q2.2 (S), C1.2, C2.2; no longer Q1.3 (S), Q2.3 (S)
- net at P1.11 (D5_PWM), R2.1: now also R4.2; no longer Q2.1 (G)
- net at P1.12 (D6_PWM), R1.1: now also R3.2; no longer Q1.1 (G)
- net at P3.2 (P2): now also Q1.3 (D); no longer Q1.2 (D)
- net at P4.2 (P2): now also Q2.3 (D); no longer Q2.2 (D)
- new net: Q1.1 (G), R3.1
- new net: Q2.1 (G), R4.1
Other:
- moved on the sheet: P2, P3, P4
Changed lines of the file:
@@
 LIBS:mysensors_mcu
 LIBS:MysXLedDimmer-cache
-EELAYER 25 0
+EELAYER 26 0
 EELAYER END
 $Descr A4 11693 8268
@@
 $EndDescr
 $Comp
-L MYSX_1.3 P1
+L MYSX_2.3 P1
 U 1 1 56C06C44
 P 4450 3300
 F 0 "P1" H 4700 3400 50  0000 C CNN
-F 1 "MYSX_1.3" H 5000 3400 50  0000 C CNN
+F 1 "MYSX_2.4" H 5000 3400 50  0000 C CNN
 F 2 "mysensors_connectors:MYSX_1.3" H 4450 2100 60  0001 C CNN
 F 3 "" H 4450 2100 60  0000 C CNN
@@
 $EndComp
 $Comp
-L Q_PMOS_GDS Q1
-U 1 1 56C06C94
-P 6300 3800
-F 0 "Q1" H 6600 3850 50  0000 R CNN
-F 1 "IRLZ44N" H 6950 3750 50  0000 R CNN
-F 2 "TO_SOT_Packages_THT:TO-220_Neutral123_Vertical" H 6500 3900 50  0001 C CNN
-F 3 "" H 6300 3800 50  0000 C CNN
-	1    6300 3800
-	1    0    0    -1
-$EndComp
-$Comp
-L Q_PMOS_GDS Q2
+L Q_NMOS_GSD Q2
 U 1 1 56C06D3D
-P 6300 4450
-F 0 "Q2" H 6600 4500 50  0000 R CNN
-F 1 "IRLZ44N" H 6950 4400 50  0000 R CNN
-F 2 "TO_SOT_Packages_THT:TO-220_Neutral123_Vertical" H 6500 4550 50  0001 C CNN
-F 3 "" H 6300 4450 50  0000 C CNN
-	1    6300 4450
-	1    0    0    -1
-$EndComp
-Wire Wire Line
-	6100 4450 4350 4450
+P 6700 4450
+F 0 "Q2" H 7000 4500 50  0000 R CNN
+F 1 "IRLML2502" H 7350 4400 50  0000 R CNN
+F 2 "TO_SOT_Packages_SMD:SOT-23_Handsoldering" H 6900 4550 50  0001 C CNN
+F 3 "" H 6700 4450 50  0000 C CNN
+	1    6700 4450
+	1    0    0    -1
+$EndComp
 Wire Wire Line
 	4350 4450 4350 3800
 Wire Wire Line
 	4350 3800 4450 3800
-Wire Wire Line
-	5500 3800 6100 3800
 $Comp
 L CONN_01X02 P3
 U 1 1 56C06E21
-P 7300 3550
-F 0 "P3" H 7300 3700 50  0000 C CNN
-F 1 "CONN_01X02" V 7400 3550 50  0000 C CNN
-F 2 "mysensors_connectors:TerminalBlock2.54mmx2-kcswalter" H 7300 3550 50  0001 C CNN
-F 3 "" H 7300 3550 50  0000 C CNN
-	1    7300 3550
-	1    0    0    -1
-$EndComp
-Wire Wire Line
-	6400 3600 7100 3600
+P 7700 3550
+F 0 "P3" H 7700 3700 50  0000 C CNN
+F 1 "CONN_01X02" V 7800 3550 50  0000 C CNN
+F 2 "mysensors_connectors:TerminalBlock2.54mmx2-kcswalter" H 7700 3550 50  0001 C CNN
+F 3 "" H 7700 3550 50  0000 C CNN
+	1    7700 3550
+	1    0    0    -1
+$EndComp
+Wire Wire Line
+	6800 3600 7500 3600
 $Comp
 L CONN_01X02 P4
 U 1 1 56C06E7D
-P 7300 4200
-F 0 "P4" H 7300 4350 50  0000 C CNN
-F 1 "CONN_01X02" V 7400 4200 50  0000 C CNN
-F 2 "mysensors_connectors:TerminalBlock2.54mmx2-kcswalter" H 7300 4200 50  0001 C CNN
-F 3 "" H 7300 4200 50  0000 C CNN
-	1    7300 4200
-	1    0    0    -1
-$EndComp
-Wire Wire Line
-	6400 4250 7100 4250
+P 7700 4200
+F 0 "P4" H 7700 4350 50  0000 C CNN
+F 1 "CONN_01X02" V 7800 4200 50  0000 C CNN
+F 2 "mysensors_connectors:TerminalBlock2.54mmx2-kcswalter" H 7700 4200 50  0001 C CNN
+F 3 "" H 7700 4200 50  0000 C CNN
+	1    7700 4200
+	1    0    0    -1
+$EndComp
+Wire Wire Line
+	6800 4250 7500 4250
 $Comp
 L GND #PWR01
 U 1 1 56C06EB9
-P 6400 4000
-F 0 "#PWR01" H 6400 3750 50  0001 C CNN
-F 1 "GND" H 6400 3850 50  0000 C CNN
-F 2 "" H 6400 4000 50  0000 C CNN
-F 3 "" H 6400 4000 50  0000 C CNN
-	1    6400 4000
+P 6800 4000
+F 0 "#PWR01" H 6800 3750 50  0001 C CNN
+F 1 "GND" H 6800 3850 50  0000 C CNN
+F 2 "" H 6800 4000 50  0000 C CNN
+F 3 "" H 6800 4000 50  0000 C CNN
+	1    6800 4000
 	1    0    0    -1
 $EndComp
@@
 L GND #PWR02
 U 1 1 56C06ED9
-P 6400 4650
-F 0 "#PWR02" H 6400 4400 50  0001 C CNN
-F 1 "GND" H 6400 4500 50  0000 C CNN
-F 2 "" H 6400 4650 50  0000 C CNN
-F 3 "" H 6400 4650 50  0000 C CNN
-	1    6400 4650
+P 6800 4650
+F 0 "#PWR02" H 6800 4400 50  0001 C CNN
+F 1 "GND" H 6800 4500 50  0000 C CNN
+F 2 "" H 6800 4650 50  0000 C CNN
+F 3 "" H 6800 4650 50  0000 C CNN
+	1    6800 4650
 	1    0    0    -1
 $EndComp
@@
 L CONN_01X02 P2
 U 1 1 56C06F52
-P 7300 2850
-F 0 "P2" H 7300 3000 50  0000 C CNN
-F 1 "CONN_01X02" V 7400 2850 50  0000 C CNN
-F 2 "mysensors_connectors:TerminalBlock2.54mmx2-kcswalter" H 7300 2850 50  0001 C CNN
-F 3 "" H 7300 2850 50  0000 C CNN
-	1    7300 2850
+P 7700 2850
+F 0 "P2" H 7700 3000 50  0000 C CNN
+F 1 "CONN_01X02" V 7800 2850 50  0000 C CNN
+F 2 "mysensors_connectors:TerminalBlock2.54mmx2-kcswalter" H 7700 2850 50  0001 C CNN
+F 3 "" H 7700 2850 50  0000 C CNN
+	1    7700 2850
 	1    0    0    -1
 $EndComp
@@
 L GND #PWR03
 U 1 1 56C06FC9
-P 7100 2900
-F 0 "#PWR03" H 7100 2650 50  0001 C CNN
-F 1 "GND" H 7100 2750 50  0000 C CNN
-F 2 "" H 7100 2900 50  0000 C CNN
-F 3 "" H 7100 2900 50  0000 C CNN
-	1    7100 2900
+P 7500 2900
+F 0 "#PWR03" H 7500 2650 50  0001 C CNN
+F 1 "GND" H 7500 2750 50  0000 C CNN
+F 2 "" H 7500 2900 50  0000 C CNN
+F 3 "" H 7500 2900 50  0000 C CNN
+	1    7500 2900
 	1    0    0    -1
 $EndComp
@@
 L +12V #PWR04
 U 1 1 56C07007
-P 7100 2750
-F 0 "#PWR04" H 7100 2600 50  0001 C CNN
-F 1 "+12V" H 7100 2890 50  0000 C CNN
-F 2 "" H 7100 2750 50  0000 C CNN
-F 3 "" H 7100 2750 50  0000 C CNN
-	1    7100 2750
-	1    0    0    -1
-$EndComp
-Wire Wire Line
-	7100 2750 7100 2800
+P 7500 2750
+F 0 "#PWR04" H 7500 2600 50  0001 C CNN
+F 1 "+12V" H 7500 2890 50  0000 C CNN
+F 2 "" H 7500 2750 50  0000 C CNN
+F 3 "" H 7500 2750 50  0000 C CNN
+	1    7500 2750
+	1    0    0    -1
+$EndComp
+Wire Wire Line
+	7500 2750 7500 2800
 $Comp
 L +12V #PWR05
 U 1 1 56C07039
-P 7100 3450
-F 0 "#PWR05" H 7100 3300 50  0001 C CNN
-F 1 "+12V" H 7100 3590 50  0000 C CNN
-F 2 "" H 7100 3450 50  0000 C CNN
-F 3 "" H 7100 3450 50  0000 C CNN
-	1    7100 3450
+P 7500 3450
+F 0 "#PWR05" H 7500 3300 50  0001 C CNN
+F 1 "+12V" H 7500 3590 50  0000 C CNN
+F 2 "" H 7500 3450 50  0000 C CNN
+F 3 "" H 7500 3450 50  0000 C CNN
+	1    7500 3450
 	1    0    0    -1
 $EndComp
@@
 L +12V #PWR06
 U 1 1 56C0705B
-P 7100 4100
-F 0 "#PWR06" H 7100 3950 50  0001 C CNN
-F 1 "+12V" H 7100 4240 50  0000 C CNN
-F 2 "" H 7100 4100 50  0000 C CNN
-F 3 "" H 7100 4100 50  0000 C CNN
-	1    7100 4100
-	1    0    0    -1
-$EndComp
-Wire Wire Line
-	7100 4100 7100 4150
-Wire Wire Line
-	7100 3450 7100 3500
+P 7500 4100
+F 0 "#PWR06" H 7500 3950 50  0001 C CNN
+F 1 "+12V" H 7500 4240 50  0000 C CNN
+F 2 "" H 7500 4100 50  0000 C CNN
+F 3 "" H 7500 4100 50  0000 C CNN
+	1    7500 4100
+	1    0    0    -1
+$EndComp
+Wire Wire Line
+	7500 4100 7500 4150
+Wire Wire Line
+	7500 3450 7500 3500
 $Comp
 L +12V #PWR07
@@
 P 5850 4000
 F 0 "R1" V 5930 4000 50  0000 C CNN
-F 1 "2k2" V 5850 4000 50  0000 C CNN
+F 1 "100k" V 5850 4000 50  0000 C CNN
 F 2 "Resistors_SMD:R_0805_HandSoldering" V 5780 4000 50  0001 C CNN
 F 3 "" H 5850 4000 50  0000 C CNN
@@
 P 5850 4650
 F 0 "R2" V 5930 4650 50  0000 C CNN
-F 1 "2k2" V 5850 4650 50  0000 C CNN
+F 1 "100k" V 5850 4650 50  0000 C CNN
 F 2 "Resistors_SMD:R_0805_HandSoldering" V 5780 4650 50  0001 C CNN
 F 3 "" H 5850 4650 50  0000 C CNN
@@
 	5850 4500 5850 4450
 Connection ~ 5850 4450
+$Comp
+L Q_NMOS_GSD Q1
+U 1 1 56C06C94
+P 6700 3800
+F 0 "Q1" H 7000 3850 50  0000 R CNN
+F 1 "IRLML2502" H 7350 3750 50  0000 R CNN
+F 2 "TO_SOT_Packages_SMD:SOT-23_Handsoldering" H 6900 3900 50  0001 C CNN
+F 3 "" H 6700 3800 50  0000 C CNN
+	1    6700 3800
+	1    0    0    -1
+$EndComp
+$Comp
+L R R4
+U 1 1 58A81E2F
+P 6200 4450
+F 0 "R4" V 5993 4450 50  0000 C CNN
+F 1 "27" V 6084 4450 50  0000 C CNN
+F 2 "Resistors_SMD:R_0805_HandSoldering" V 30  0   50  0001 C CNN
+F 3 "" H 100 0   50  0001 C CNN
+	1    6200 4450
+	0    1    1    0
+$EndComp
+$Comp
+L R R3
+U 1 1 58A81ECB
+P 6200 3800
+F 0 "R3" V 5993 3800 50  0000 C CNN
+F 1 "27" V 6084 3800 50  0000 C CNN
+F 2 "Resistors_SMD:R_0805_HandSoldering" V -70 -100 50  0001 C CNN
+F 3 "" H 0   -100 50  0001 C CNN
+	1    6200 3800
+	0    1    1    0
+$EndComp
+Wire Wire Line
+	6350 4450 6500 4450
+Wire Wire Line
+	6350 3800 6500 3800
+Wire Wire Line
+	5500 3800 6050 3800
+Wire Wire Line
+	4350 4450 6050 4450
+$Comp
+L CP C2
+U 1 1 58A8219F
+P 4000 3500
+F 0 "C2" H 4118 3546 50  0000 L CNN
+F 1 "CP" H 4118 3455 50  0000 L CNN
+F 2 "Capacitors_SMD:C_0805_HandSoldering" H -1912 100 50  0001 C CNN
+F 3 "" H -1950 250 50  0001 C CNN
+	1    4000 3500
+	1    0    0    -1
+$EndComp
+$Comp
+L C C1
+U 1 1 58A8225E
+P 3650 3500
+F 0 "C1" H 3765 3546 50  0000 L CNN
+F 1 "C" H 3765 3455 50  0000 L CNN
+F 2 "Capacitors_SMD:C_0805_HandSoldering" H -362 0   50  0001 C CNN
+F 3 "" H -400 150 50  0001 C CNN
+	1    3650 3500
+	1    0    0    -1
+$EndComp
+Wire Wire Line
+	3650 3350 4000 3350
+Wire Wire Line
+	3650 3650 4000 3650
+$Comp
+L GND #PWR011
+U 1 1 58A822EB
+P 3800 3850
+F 0 "#PWR011" H 0   -150 50  0001 C CNN
+F 1 "GND" H 3805 3677 50  0000 C CNN
+F 2 "" H 0   100 50  0001 C CNN
+F 3 "" H 0   100 50  0001 C CNN
+	1    3800 3850
+	1    0    0    -1
+$EndComp
+Wire Wire Line
+	3800 3850 3800 3650
+Connection ~ 3800 3650
+Wire Wire Line
+	3800 3350 3800 3300
+Wire Wire Line
+	3800 3300 4450 3300
+Connection ~ 3800 3350
 $EndSCHEMATC
